File: pulse eagle/pulse sensor.sch (EAGLE design)
At the start: 8 parts

Commit message: Revision 2 of the pulse sensor. Upgrading to tantalum cap, switching the two caps, and using the correct resistor value. Also switching to temrinal connectors on bottom of board.
Parts:
- C2: value 15uF -> 22uF; device SparkFun-Capacitors:10UF-6.3V-20%(0603) -> SparkFun-Passives:CAP_POL1206
- R1: value 1.5k -> 30
- SL2: device SparkFun-Connectors:M04POLAR_LOCK -> SparkFun-Connectors:M04SMD
Connections:
- net 3V3: now also C1.1; no longer C2.1
- net GND: now also C2.-; no longer C2.2
- net N$2: now also C2.+; no longer C1.1
Other:
- moved on the sheet: C1
Changed lines of the file:
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@@
 <?xml version="1.0" encoding="utf-8"?>
 <!DOCTYPE eagle SYSTEM "eagle.dtd">
-<eagle version="6.6.0">
+<eagle version="7.0.0">
 <drawing>
 <settings>
@@
 <parts>
 <part name="LED1" library="SparkFun-LED" deviceset="LED" device="1206"/>
-<part name="R1" library="resistor" deviceset="R-US_" device="R0402" value="1.5k"/>
+<part name="R1" library="resistor" deviceset="R-US_" device="R0402" value="30"/>
 <part name="U$2" library="pulse" deviceset="SI1143" device=""/>
 <part name="LED2" library="SparkFun-LED" deviceset="LED" device="1206"/>
 <part name="LED3" library="SparkFun-LED" deviceset="LED" device="1206"/>
 <part name="C1" library="SparkFun-Capacitors" deviceset=".1UF-CER" device="" value="0.1uF"/>
-<part name="SL2" library="SparkFun-Connectors" deviceset="M04" device="POLAR_LOCK"/>
-<part name="C2" library="SparkFun-Capacitors" deviceset="10UF-6.3V-20%(0603)" device="" value="15uF"/>
+<part name="SL2" library="SparkFun-Connectors" deviceset="M04" device="SMD"/>
+<part name="C2" library="SparkFun-Passives" deviceset="CAP_POL" device="1206" value="22uF"/>
 </parts>
 <sheets>
@@
 <instance part="LED2" gate="G$1" x="81.28" y="45.72" rot="R270"/>
 <instance part="LED3" gate="G$1" x="81.28" y="55.88" rot="R270"/>
-<instance part="C1" gate="G$1" x="99.06" y="38.1"/>
+<instance part="C1" gate="G$1" x="109.22" y="45.72"/>
 <instance part="SL2" gate="G$1" x="129.54" y="45.72"/>
-<instance part="C2" gate="G$1" x="109.22" y="45.72"/>
+<instance part="C2" gate="G$1" x="99.06" y="40.64"/>
 </instances>
 <busses>
@@
 <segment>
 <pinref part="R1" gate="G$1" pin="2"/>
-<pinref part="C1" gate="G$1" pin="1"/>
 <wire x1="99.06" y1="48.26" x2="99.06" y2="45.72" width="0.1524" layer="91"/>
 <pinref part="LED2" gate="G$1" pin="A"/>
-<wire x1="99.06" y1="45.72" x2="99.06" y2="43.18" width="0.1524" layer="91"/>
 <wire x1="99.06" y1="45.72" x2="88.9" y2="45.72" width="0.1524" layer="91"/>
-<junction x="99.06" y="45.72"/>
 <wire x1="88.9" y1="45.72" x2="83.82" y2="45.72" width="0.1524" layer="91"/>
 <wire x1="88.9" y1="45.72" x2="88.9" y2="35.56" width="0.1524" layer="91"/>
@@
 <pinref part="LED3" gate="G$1" pin="A"/>
 <wire x1="88.9" y1="55.88" x2="83.82" y2="55.88" width="0.1524" layer="91"/>
+<wire x1="99.06" y1="45.72" x2="99.06" y2="43.18" width="0.1524" layer="91"/>
+<junction x="99.06" y="45.72"/>
+<pinref part="C2" gate="G$1" pin="+"/>
 </segment>
 </net>
@@
 </segment>
 <segment>
-<pinref part="C1" gate="G$1" pin="2"/>
-<wire x1="99.06" y1="35.56" x2="99.06" y2="33.02" width="0.1524" layer="91"/>
 <wire x1="99.06" y1="33.02" x2="109.22" y2="33.02" width="0.1524" layer="91"/>
 <label x="111.76" y="33.02" size="1.016" layer="95" xref="yes"/>
-<pinref part="C2" gate="G$1" pin="2"/>
 <wire x1="109.22" y1="33.02" x2="111.76" y2="33.02" width="0.1524" layer="91"/>
+<wire x1="99.06" y1="35.56" x2="99.06" y2="33.02" width="0.1524" layer="91"/>
+<pinref part="C1" gate="G$1" pin="2"/>
 <wire x1="109.22" y1="43.18" x2="109.22" y2="33.02" width="0.1524" layer="91"/>
 <junction x="109.22" y="33.02"/>
+<pinref part="C2" gate="G$1" pin="-"/>
 </segment>
 <segment>
@@
 <wire x1="99.06" y1="60.96" x2="109.22" y2="60.96" width="0.1524" layer="91"/>
 <label x="111.76" y="60.96" size="1.016" layer="95" xref="yes"/>
-<pinref part="C2" gate="G$1" pin="1"/>
+<pinref part="C1" gate="G$1" pin="1"/>
 <wire x1="109.22" y1="60.96" x2="111.76" y2="60.96" width="0.1524" layer="91"/>
 <wire x1="109.22" y1="60.96" x2="109.22" y2="50.8" width="0.1524" layer="91"/>
